File: Arm_Mainboard/RoboticArmActuators.sch (KiCad schematic (older format))
At the start: 0 parts

Commit message: PCB
Parts:
- added A1, A2, A3: Pololu_Breakout_A4988, ArmFootprints:Pololu_Breakout-16_15.2x20.3mm, symbol Driver_Motor:Pololu_Breakout_A4988
- added C22, C23, C24: 100uF, Capacitor_SMD:CP_Elec_8x10, symbol Device:CP1
- added J11, J13, J15, J21, J23, J25: 12V, Jumper:SolderJumper-2_P1.3mm_Open_RoundedPad1.0x1.5mm, symbol Connector:Conn_01x02_Male
- added J14, J22, J26: CONN, Connector_JST:JST_EH_S4B-EH_1x04_P2.50mm_Horizontal, symbol Connector:Conn_01x04_Male
- added J16: CONN_NEMA23_2, Connector_JST:JST_EH_S4B-EH_1x04_P2.50mm_Horizontal, symbol Connector:Conn_01x04_Male
- added J18: CONN_NEMA23_1, Connector_JST:JST_EH_S4B-EH_1x04_P2.50mm_Horizontal, symbol Connector:Conn_01x04_Male
- added J19: NEMA23_2, ArmFootprints:Molex_12PIN, symbol Connector:Conn_01x12_Male
- added J20: NEMA23_1, ArmFootprints:Molex_12PIN, symbol Connector:Conn_01x12_Male
- added S1, S2, S3: DIP SWITCH, ArmFootprints:SW_DS04-254-2-03BK-SMT, symbol DS04-254-2-03BK-SMT:DS04-254-2-03BK-SMT
Connections:
- new net: J18.1 (Pin_1), J20.10 (Pin_10)
- new net: J18.4 (Pin_4), J20.7 (Pin_7)
- new net: J18.3 (Pin_3), J20.8 (Pin_8)
- new net: J18.2 (Pin_2), J20.9 (Pin_9)
- new net: J16.1 (Pin_1), J19.10 (Pin_10)
- new net: J16.4 (Pin_4), J19.7 (Pin_7)
- new net: J16.3 (Pin_3), J19.8 (Pin_8)
- new net: J16.2 (Pin_2), J19.9 (Pin_9)
- new net: A1.6 (2B), J14.1 (Pin_1)
- new net: A1.5 (2A), J14.2 (Pin_2)
- new net: A1.4 (1A), J14.3 (Pin_3)
- new net: A1.3 (1B), J14.4 (Pin_4)
- new net: A1.13 (~RESET), A1.14 (~SLEEP)
- new net: A2.6 (2B), J22.1 (Pin_1)
- new net: A2.5 (2A), J22.2 (Pin_2)
- new net: A2.4 (1A), J22.3 (Pin_3)
- new net: A2.3 (1B), J22.4 (Pin_4)
- new net: A2.13 (~RESET), A2.14 (~SLEEP)
- new net: A3.6 (2B), J26.1 (Pin_1)
- new net: A3.5 (2A), J26.2 (Pin_2)
- new net: A3.4 (1A), J26.3 (Pin_3)
- new net: A3.3 (1B), J26.4 (Pin_4)
- new net: A3.13 (~RESET), A3.14 (~SLEEP)
- new net +12V: J11.1 (Pin_1), J15.1 (Pin_1), J19.12 (Pin_12), J20.12 (Pin_12), J23.1 (Pin_1)
- new net DIR-NEMA11: A3.16 (DIR)
- new net DIR-NEMA14_1: A1.16 (DIR)
- new net DIR-NEMA14_2: A2.16 (DIR)
- new net DIR-NEMA23_1: J20.4 (Pin_4)
- new net DIR-NEMA23_2: J19.4 (Pin_4)
- new net GND: A1.1 (GND), A1.7 (GND), A2.1 (GND), A2.7 (GND), A3.1 (GND), A3.7 (GND), C22.2, C23.2, C24.2, J19.11 (Pin_11), J19.3 (Pin_3), J19.5 (Pin_5), J20.11 (Pin_11), J20.3 (Pin_3), J20.5 (Pin_5)
- new net MS1-NEMA11: A3.10 (MS1), S3.1B
- new net MS1-NEMA14_1: A1.10 (MS1), S1.1B
- new net MS1-NEMA14_2: A2.10 (MS1), S2.1B
- new net MS2-NEMA11: A3.11 (MS2), S3.2B
- new net MS2-NEMA14_1: A1.11 (MS2), S1.2B
- new net MS2-NEMA14_2: A2.11 (MS2), S2.2B
- new net MS3-NEMA11: A3.12 (MS3), S3.3B
- new net MS3-NEMA14_1: A1.12 (MS3), S1.3B
- new net MS3-NEMA14_2: A2.12 (MS3), S2.3B
- new net STEP-NEMA11: A3.15 (STEP)
- new net STEP-NEMA14_1: A1.15 (STEP)
- new net STEP-NEMA14_2: A2.15 (STEP)
- new net STEP-NEMA23_1: J20.6 (Pin_6)
- new net STEP-NEMA23_2: J19.6 (Pin_6)
- new net VDD5: A1.2 (VDD), A2.2 (VDD), A3.2 (VDD), J13.1 (Pin_1), J21.1 (Pin_1), J25.1 (Pin_1), S1.1A, S1.2A, S1.3A, S2.1A, S2.2A, S2.3A, S3.1A, S3.2A, S3.3A
- new net V_MOT: A1.8 (VMOT), A2.8 (VMOT), A3.8 (VMOT), C22.1, C23.1, C24.1, J11.2 (Pin_2), J13.2 (Pin_2), J15.2 (Pin_2), J21.2 (Pin_2), J23.2 (Pin_2), J25.2 (Pin_2)
- no-connect marks 0 -> 7
Other:
- note added: "AXIS 1 [NEMA23]\n"
- note added: "AXIS 2 [NEMA23]\n"
- note added: "AXIS 3 [NEMA14]\n"
- note added: "AXIS 4 [NEMA14]\n"
- note added: "AXIS 5 [NEMA11]\n"
