File: Arm_Mainboard/Arm_Mainboard.kicad_pcb (KiCad board)
At the start: 2 copper layers, 163.4 x 100.6 mm, 113 parts, among them J10 FAN HEADER 2, J14 CONN, J16 CONN_NEMA23_2, J19 NEMA23_2, J2 JTAG, J20 NEMA23_1, J22 CONN, J26 CONN, J27 ENC_AXIS1, J28 ENC_AXIS2, J29 ENC_AXIS3, J30 ENC_AXIS4, J31 ENC_AXIS5, J4 USB PINOUT, J6 UART, J7 BOOT OPTION, J8 POWER, J9 FAN HEADER 1, Q1 P_CH MOSFET, U1 ESP32-WROOM-32U, U2 MCP2200-I-SS, U3 LM2678SX-3.3/NOPB, U4 LM2678S-5.0/NOPB, Y1 Resonator

Commit message: gerbers
Parts:
- removed the G*** at (204.2, 122.2)
- added G***: LOGO, logos:QRcode_Smaller, B.Cu at (202.8, 121.5)
